File: ADS1115-Breakout-5V.brd (EAGLE design)
At the start: 27.9 x 17.1 mm, 22 parts, among them IC2 MCP1703CB, U1 ADS1115IDGST

Commit message: Some trace & silkscreen adjustments
Parts:
- moved R10 0.63 mm to (10.5, 11.6)
- moved R2 0.63 mm to (9.14, 11.6)
- moved Q1 0.44 mm to (7.81, 8.57)
- moved Q3 0.44 mm to (11.9, 8.57)
- moved R1 0.44 mm to (9.14, 9.46)
- moved R9 0.44 mm to (10.5, 9.46)
Routing:
- net GND: track 14.8 -> 23.4 mm
- net SDA_3V3: track 9.47 -> 10.6 mm
- net 3V3: track 23.0 -> 22.1 mm
- net SCL_5V: track 27.9 -> 27.1 mm
- net SDA_5V: track 22.1 -> 21.2 mm
Other:
- board text added: "ADS1115 0-5V input 3.3V I2C"
- board text removed: "ADS1115"
